File: schematics/relayBoard.brd (EAGLE design)
At the start: 94.9 x 69.8 mm, 21 parts, among them K1 AQG12105, K2 AQG12105

Commit message: board and schematics work in progress
Parts:
- removed AC-OUT-1, AC-OUT-2: (no value), con-wago-500:W237-102
- added CONN-SW: (no value), con-wago-500:W237-103
- C1, C2: value (none) -> 0.1uF; device resistor:PANASONIC_C -> SparkFun-Capacitors:0603-CAP
- moved AC-IN 61.6 mm to (73.7, 10.2), turned to 270 degrees
- moved R6 33.2 mm to (11.4, 31.8), turned to 90 degrees
- moved JP3 30.7 mm to (17.8, 3.81)
- moved R3 30.7 mm to (8.89, 31.8), turned to 90 degrees
- moved C1 30.2 mm to (30.5, 10.2), turned to 270 degrees
- moved U$4 30.2 mm to (67.3, 20.3)
- moved R7 25.3 mm to (12.7, 5.08), turned to 270 degrees
- moved R2 25.0 mm to (8.89, 5.08), turned to 90 degrees
- moved R5 24.7 mm to (5.08, 5.08), turned to 90 degrees
- moved U$1 23.2 mm to (24.1, 10.2)
- moved R8 22.2 mm to (20.3, 7.62), turned to 0 degrees
- moved R4 21.6 mm to (24.1, 29.2)
- moved C2 20.9 mm to (27.9, 26.7), turned to 90 degrees
- moved JP1 19.7 mm to (20.3, 31.8), turned to 180 degrees
- moved K1 15.5 mm to (55.9, 24.1), turned to 0 degrees
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Connections:
- removed net AC-L: AC-IN.2, K1.O1, K2.O1, U$4.AC2
- removed net AC-N: AC-IN.1, AC-OUT-1.2, AC-OUT-2.2, U$4.AC1
- new net AC-SW-L: CONN-SW.1, K1.O1, K2.O1
- new net N$2: AC-IN.1, U$4.AC2
- new net N$5: AC-IN.2, U$4.AC1
- net 3V3: now also C2.1, R7.2, R8.2; no longer C2.+
- net 5V: now also C1.1; no longer C1.+
- net GND: now also C1.2, C2.2; no longer C1.-, C2.-
- net LOAD1: now also CONN-SW.2; no longer AC-OUT-1.1
- net LOAD2: now also CONN-SW.3; no longer AC-OUT-2.1
Routing:
- net GND: track 0.00 -> 121.4 mm
- net 3V3: track 0.00 -> 66.6 mm
- net AC-SW-L: track 0.00 -> 26.1 mm
- net 5V: track 0.00 -> 16.5 mm
- net RXD: track 0.00 -> 9.64 mm
- net GPIO14: track 0.00 -> 9.56 mm
- net LOAD2: track 0.00 -> 9.45 mm
- net LOAD1: track 0.00 -> 9.41 mm
- net GPIO16: track 0.00 -> 8.69 mm
- net N$5: track 0.00 -> 7.41 mm
- net N$2: track 0.00 -> 7.41 mm
- net GPIO4: track 0.00 -> 6.09 mm
- net GPIO5: track 0.00 -> 5.56 mm
- net CH_PD: track 0.00 -> 5.42 mm
- net N$4: track 0.00 -> 5.39 mm
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Other:
- board size 94.9 x 69.8 mm -> 79.7 x 69.8 mm

Commit message: code and schematic modifications
Parts:
- added D1, D2: (no value), SparkFun-DiscreteSemi:SMA-DIODE
- added Q1, Q2: (no value), semicon-smd-ipc:SOT23
- moved R3 33.6 mm to (41.9, 38.1), turned to 0 degrees
- moved R6 30.5 mm to (41.9, 30.5), turned to 0 degrees
- moved U$4 19.9 mm to (76.2, 2.54), flipped to the bottom, turned to 0 degrees
- moved CONN-SW 18.2 mm to (91.4, 29.2), turned to 270 degrees
- moved AC-IN 16.7 mm to (90.2, 12.7)
- moved K1 13.7 mm to (63.5, 35.6), flipped to the bottom, turned to 180 degrees
- moved C1 10.2 mm to (39.4, 15.2), turned to 90 degrees
- moved U2 9.67 mm to (30.5, 16.5), turned to 180 degrees
- moved JP1 8.98 mm to (19.1, 40.6)
- moved K2 8.03 mm to (63.5, 29.2), flipped to the bottom, turned to 180 degrees
- moved R4 8.03 mm to (21.6, 36.8), turned to 270 degrees
- moved R5 2.84 mm to (7.62, 6.35)
- moved R2 2.84 mm to (11.4, 6.35)
- moved C2 2.54 mm to (27.9, 24.1)
- moved JP3 2.54 mm to (20.3, 3.81)
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Connections:
- new net N$10: D1.A, K1.-, Q1.3
- new net N$12: Q1.1, R3.2
- new net N$7: D2.A, K2.-, Q2.3
- new net N$8: Q2.1, R6.2
- net 3V3: now also D1.C, D2.C; no longer R3.2, R6.2
- net GND: now also Q1.2, Q2.2
- net GPIO4: no longer K1.-
- net GPIO5: no longer K2.-
- net N$2: now also U$4.AC1; no longer U$4.AC2
- net N$5: now also U$4.AC2; no longer U$4.AC1
Routing:
- net GND: track 121.4 -> 53.9 mm
- net 3V3: track 66.6 -> 39.6 mm
- net AC-SW-L: track 26.1 -> 0.00 mm
- net 5V: track 16.5 -> 0.00 mm
- net RXD: track 9.64 -> 0.00 mm
- net LOAD2: track 9.45 -> 0.00 mm
- net LOAD1: track 9.41 -> 0.00 mm
- net N$5: track 7.41 -> 0.00 mm
- net N$2: track 7.41 -> 0.00 mm
- net GPIO4: track 6.09 -> 0.00 mm
- net GPIO5: track 5.56 -> 0.00 mm
- net TXD: track 5.20 -> 0.00 mm
- net GPIO16: track 8.69 -> 9.87 mm
- net CH_PD: track 5.42 -> 4.68 mm
- net GPIO14: track 9.56 -> 10.3 mm
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Other:
- board size 79.7 x 69.8 mm -> 100 x 80 mm
