File: schematics/relayBoard.sch (EAGLE design)
At the start: 21 parts, among them K1 AQG12105, K2 AQG12105

Commit message: board and schematics work in progress
Parts:
- removed AC-OUT-1, AC-OUT-2: (no value), con-wago-500:W237-102
- added CONN-SW: (no value), con-wago-500:W237-103
- C1, C2: value (none) -> 0.1uF; device resistor:CPOL-EUC -> SparkFun-Capacitors:0.1UF-25V-5%(0603)
Connections:
- removed net AC-L: AC-IN-2.KL, K1.DS2, K2.DS2, U$4.AC2
- removed net AC-N: AC-IN-1.KL, AC-OUT-1-2.KL, AC-OUT-2-2.KL, U$4.AC1
- new net AC-SW-L: CONN-SW-1.KL, K1.DS2, K2.DS2
- new net N$2: AC-IN-1.KL, U$4.AC2
- new net N$5: AC-IN-2.KL, U$4.AC1
- net 3V3: now also C2.1, R7.2, R8.2; no longer C2.+
- net 5V: now also C1.1; no longer C1.+
- net GND: now also C1.2, C2.2; no longer C1.-, C2.-
- net LOAD1: now also CONN-SW-2.KL; no longer AC-OUT-1-1.KL
- net LOAD2: now also CONN-SW-3.KL; no longer AC-OUT-2-1.KL
Other:
- moved on the sheet: AC-IN-1, AC-IN-2
Changed lines of the file:
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@@
 </variantdefs>
 <classes>
-<class number="0" name="default" width="0" drill="0">
+<class number="0" name="default" width="0.1524" drill="0.3048">
+<clearance class="0" value="0.1524"/>
+</class>
+<class number="1" name="ac" width="1.27" drill="1.27">
+<clearance class="1" value="2.54"/>
 </class>
 </classes>
@@
 <part name="R3" library="resistor" deviceset="R-EU_" device="R0805" value="10K"/>
 <part name="U$4" library="hlk-pm01" deviceset="HLK-PM01" device=""/>
-<part name="C1" library="resistor" deviceset="CPOL-EU" device="C"/>
-<part name="C2" library="resistor" deviceset="CPOL-EU" device="C"/>
 <part name="JP1" library="pinhead" deviceset="PINHD-1X3" device=""/>
 <part name="R4" library="resistor" deviceset="R-EU_" device="R0805" value="10K"/>
@@
 <part name="R7" library="resistor" deviceset="R-EU_" device="R0805"/>
 <part name="R8" library="resistor" deviceset="R-EU_" device="R0805"/>
-<part name="AC-OUT-2" library="con-wago-500" deviceset="W237-102" device=""/>
-<part name="AC-OUT-1" library="con-wago-500" deviceset="W237-102" device=""/>
 <part name="AC-IN" library="con-wago-500" deviceset="W237-102" device=""/>
+<part name="C1" library="SparkFun-Capacitors" deviceset="0.1UF-25V-5%(0603)" device="" value="0.1uF"/>
+<part name="C2" library="SparkFun-Capacitors" deviceset="0.1UF-25V-5%(0603)" device="" value="0.1uF"/>
+<part name="CONN-SW" library="con-wago-500" deviceset="W237-103" device=""/>
 </parts>
 <sheets>
@@
 <instance part="R3" gate="G$1" x="109.22" y="55.88" rot="R90"/>
 <instance part="U$4" gate="G$1" x="30.48" y="25.4"/>
-<instance part="C1" gate="G$1" x="38.1" y="10.16"/>
-<instance part="C2" gate="G$1" x="60.96" y="10.16"/>
 <instance part="JP1" gate="A" x="73.66" y="76.2" rot="R180"/>
 <instance part="R4" gate="G$1" x="83.82" y="73.66"/>
@@
 <instance part="R7" gate="G$1" x="5.08" y="96.52"/>
 <instance part="R8" gate="G$1" x="5.08" y="81.28"/>
-<instance part="AC-OUT-2" gate="-1" x="157.48" y="12.7" rot="R90"/>
-<instance part="AC-OUT-2" gate="-2" x="162.56" y="12.7" rot="R90"/>
-<instance part="AC-OUT-1" gate="-1" x="114.3" y="12.7" rot="R90"/>
-<instance part="AC-OUT-1" gate="-2" x="119.38" y="12.7" rot="R90"/>
-<instance part="AC-IN" gate="-1" x="10.16" y="30.48"/>
-<instance part="AC-IN" gate="-2" x="10.16" y="25.4"/>
+<instance part="AC-IN" gate="-1" x="12.7" y="25.4"/>
+<instance part="AC-IN" gate="-2" x="12.7" y="30.48"/>
+<instance part="C1" gate="G$1" x="38.1" y="7.62"/>
+<instance part="C2" gate="G$1" x="66.04" y="7.62"/>
+<instance part="CONN-SW" gate="-1" x="109.22" y="12.7" rot="R90"/>
+<instance part="CONN-SW" gate="-2" x="114.3" y="12.7" rot="R90"/>
+<instance part="CONN-SW" gate="-3" x="157.48" y="12.7" rot="R90"/>
 </instances>
 <busses>
@@
 <segment>
 <pinref part="R2" gate="G$1" pin="1"/>
-<wire x1="17.78" y1="63.5" x2="15.24" y2="63.5" width="0.1524" layer="91"/>
 <label x="12.7" y="63.5" size="1.778" layer="95"/>
 <pinref part="R5" gate="G$1" pin="1"/>
-<wire x1="15.24" y1="63.5" x2="12.7" y2="63.5" width="0.1524" layer="91"/>
+<wire x1="17.78" y1="63.5" x2="12.7" y2="63.5" width="0.1524" layer="91"/>
 <wire x1="17.78" y1="63.5" x2="17.78" y2="68.58" width="0.1524" layer="91"/>
 <label x="12.7" y="68.58" size="1.778" layer="95"/>
-<wire x1="20.32" y1="63.5" x2="15.24" y2="63.5" width="0.1524" layer="91"/>
 <label x="12.7" y="96.52" size="1.778" layer="95"/>
+<junction x="17.78" y="63.5"/>
 </segment>
 <segment>
@@
 <wire x1="109.22" y1="60.96" x2="114.3" y2="60.96" width="0.1524" layer="91"/>
 <wire x1="114.3" y1="60.96" x2="114.3" y2="50.8" width="0.1524" layer="91"/>
-</segment>
-<segment>
-<wire x1="58.42" y1="12.7" x2="60.96" y2="12.7" width="0.1524" layer="91"/>
+<junction x="114.3" y="50.8"/>
+</segment>
+<segment>
 <label x="63.5" y="12.7" size="1.778" layer="95"/>
-<pinref part="C2" gate="G$1" pin="+"/>
-<wire x1="60.96" y1="12.7" x2="66.04" y2="12.7" width="0.1524" layer="91"/>
-<junction x="60.96" y="12.7"/>
+<wire x1="58.42" y1="12.7" x2="66.04" y2="12.7" width="0.1524" layer="91"/>
 <pinref part="U2" gate="G$1" pin="OUT"/>
+<pinref part="C2" gate="G$1" pin="1"/>
 </segment>
 <segment>
@@
 <wire x1="152.4" y1="60.96" x2="157.48" y2="60.96" width="0.1524" layer="91"/>
 <wire x1="157.48" y1="60.96" x2="157.48" y2="50.8" width="0.1524" layer="91"/>
+<junction x="157.48" y="50.8"/>
 </segment>
 <segment>
 <wire x1="12.7" y1="96.52" x2="10.16" y2="96.52" width="0.1524" layer="91"/>
+<pinref part="R7" gate="G$1" pin="2"/>
 </segment>
 <segment>
 <wire x1="12.7" y1="81.28" x2="10.16" y2="81.28" width="0.1524" layer="91"/>
 <label x="12.7" y="81.28" size="1.778" layer="95"/>
+<pinref part="R8" gate="G$1" pin="2"/>
 </segment>
 </net>
@@
 </segment>
 <segment>
-<wire x1="60.96" y1="5.08" x2="50.8" y2="5.08" width="0.1524" layer="91"/>
+<wire x1="66.04" y1="5.08" x2="50.8" y2="5.08" width="0.1524" layer="91"/>
 <wire x1="50.8" y1="5.08" x2="38.1" y2="5.08" width="0.1524" layer="91"/>
-<wire x1="66.04" y1="5.08" x2="60.96" y2="5.08" width="0.1524" layer="91"/>
 <label x="40.64" y="5.08" size="1.778" layer="95"/>
-<pinref part="C1" gate="G$1" pin="-"/>
-<pinref part="C2" gate="G$1" pin="-"/>
-<junction x="60.96" y="5.08"/>
 <pinref part="U2" gate="G$1" pin="ADJ"/>
 <junction x="50.8" y="5.08"/>
+<pinref part="C1" gate="G$1" pin="2"/>
+<pinref part="C2" gate="G$1" pin="2"/>
 </segment>
 <segment>
@@
 <wire x1="43.18" y1="12.7" x2="38.1" y2="12.7" width="0.1524" layer="91"/>
 <label x="38.1" y="12.7" size="1.778" layer="95"/>
-<pinref part="C1" gate="G$1" pin="+"/>
 <pinref part="U2" gate="G$1" pin="IN"/>
-</segment>
-</net>
-<net name="AC-N" class="0">
-<segment>
-<label x="119.38" y="20.32" size="1.778" layer="95" rot="R90"/>
-<wire x1="119.38" y1="17.78" x2="119.38" y2="25.4" width="0.1524" layer="91"/>
-<pinref part="AC-OUT-1" gate="-2" pin="KL"/>
-</segment>
-<segment>
-<pinref part="U$4" gate="G$1" pin="AC1"/>
-<wire x1="15.24" y1="30.48" x2="30.48" y2="30.48" width="0.1524" layer="91"/>
-<label x="15.24" y="30.48" size="1.778" layer="95"/>
-<pinref part="AC-IN" gate="-1" pin="KL"/>
-</segment>
-<segment>
-<label x="162.56" y="20.32" size="1.778" layer="95" rot="R90"/>
-<wire x1="162.56" y1="17.78" x2="162.56" y2="25.4" width="0.1524" layer="91"/>
-<pinref part="AC-OUT-2" gate="-2" pin="KL"/>
-</segment>
-</net>
-<net name="AC-L" class="0">
-<segment>
-<pinref part="K1" gate="A" pin="DS2"/>
-<wire x1="109.22" y1="27.94" x2="109.22" y2="20.32" width="0.1524" layer="91"/>
-<label x="109.22" y="20.32" size="1.778" layer="95" rot="R90"/>
-</segment>
-<segment>
-<label x="15.24" y="25.4" size="1.778" layer="95"/>
-<pinref part="U$4" gate="G$1" pin="AC2"/>
-<wire x1="15.24" y1="25.4" x2="30.48" y2="25.4" width="0.1524" layer="91"/>
-<pinref part="AC-IN" gate="-2" pin="KL"/>
-</segment>
-<segment>
-<pinref part="K2" gate="A" pin="DS2"/>
-<wire x1="152.4" y1="27.94" x2="152.4" y2="20.32" width="0.1524" layer="91"/>
-<label x="152.4" y="20.32" size="1.778" layer="95" rot="R90"/>
-</segment>
-</net>
-<net name="LOAD1" class="0">
+<pinref part="C1" gate="G$1" pin="1"/>
+</segment>
+</net>
+<net name="LOAD1" class="1">
 <segment>
 <pinref part="K1" gate="A" pin="DS1"/>
 <wire x1="114.3" y1="27.94" x2="114.3" y2="17.78" width="0.1524" layer="91"/>
 <label x="114.3" y="20.32" size="1.778" layer="95" rot="R90"/>
-<pinref part="AC-OUT-1" gate="-1" pin="KL"/>
+<pinref part="CONN-SW" gate="-2" pin="KL"/>
 </segment>
 </net>
@@
 </segment>
 </net>
-<net name="LOAD2" class="0">
+<net name="LOAD2" class="1">
 <segment>
 <pinref part="K2" gate="A" pin="DS1"/>
 <wire x1="157.48" y1="27.94" x2="157.48" y2="17.78" width="0.1524" layer="91"/>
-<pinref part="AC-OUT-2" gate="-1" pin="KL"/>
 <label x="157.48" y="20.32" size="1.778" layer="95" rot="R90"/>
+<pinref part="CONN-SW" gate="-3" pin="KL"/>
 </segment>
 </net>
@@
 </segment>
 </net>
+<net name="AC-SW-L" class="1">
+<segment>
+<pinref part="K1" gate="A" pin="DS2"/>
+<wire x1="109.22" y1="27.94" x2="109.22" y2="17.78" width="0.1524" layer="91"/>
+<label x="109.22" y="20.32" size="1.778" layer="95" rot="R90"/>
+<pinref part="CONN-SW" gate="-1" pin="KL"/>
+</segment>
+<segment>
+<pinref part="K2" gate="A" pin="DS2"/>
+<wire x1="152.4" y1="27.94" x2="152.4" y2="20.32" width="0.1524" layer="91"/>
+<label x="152.4" y="20.32" size="1.778" layer="95" rot="R90"/>
+</segment>
+</net>
+<net name="N$2" class="1">
+<segment>
+<pinref part="AC-IN" gate="-1" pin="KL"/>
+<pinref part="U$4" gate="G$1" pin="AC2"/>
+<wire x1="17.78" y1="25.4" x2="30.48" y2="25.4" width="0.1524" layer="91"/>
+</segment>
+</net>
+<net name="N$5" class="1">
+<segment>
+<pinref part="AC-IN" gate="-2" pin="KL"/>
+<pinref part="U$4" gate="G$1" pin="AC1"/>
+<wire x1="17.78" y1="30.48" x2="30.48" y2="30.48" width="0.1524" layer="91"/>
+</segment>
+</net>

Commit message: code and schematic modifications
Parts:
- added D1, D2: (no value), SparkFun-DiscreteSemi:DIODESMA
- added Q1, Q2: (no value), semicon-smd-ipc:NPN-TRANSISTOR_SOT23
Connections:
- new net N$10: D1.A, K1.K, Q1.C
- new net N$12: Q1.B, R3.2
- new net N$7: D2.A, K2.K, Q2.C
- new net N$8: Q2.B, R6.2
- net 3V3: now also D1.C, D2.C; no longer R3.2, R6.2
- net GND: now also Q1.E, Q2.E
- net GPIO4: no longer K1.K
- net GPIO5: no longer K2.K
- net N$2: now also U$4.AC1; no longer U$4.AC2
- net N$5: now also U$4.AC2; no longer U$4.AC1
Other:
- moved on the sheet: AC-IN-1, AC-IN-2, JP1, JP2, R1, R3, R4, R6
