File: schematics/2ssrSingleSide/relayBoard.sch (EAGLE design)
At the start: 24 parts, among them K1 AQG12105, K2 AQG12105

Commit message: moved schematics and board
Parts:
- removed U$1: ESP8266_ESP-12, ESP8266-ESP12:ESP8266_ESP-12
- added MDL1: (no value), ESP8266-ESP12E:ESP8266-12EESP8266-ESP12E
Connections:
- removed net AC-SW-L: CONN-SW-1.KL, K1.DS2, K2.DS2
- removed net CH_PD: R2.2, U$1.CH_PD
- removed net GPIO2: U$1.GPIO2
- removed net LOAD1: CONN-SW-2.KL, K1.DS1
- removed net LOAD2: CONN-SW-3.KL, K2.DS1
- removed net N$4: R5.2, U$1.REST
- new net LOAD1L: CONN-SW-1.KL, K1.DS1
- new net LOAD2L: CONN-SW-2.KL, K2.DS1
- new net LOADN: CONN-SW-3.KL, K1.DS2, K2.DS2
- new net N$6: MDL1.REST, R5.2
- new net N$9: MDL1.CH_PD, R2.2
- net 3V3: now also MDL1.VCC; no longer D1.C, D2.C, K1.A, K2.A, U$1.VCC
- net 5V: now also D1.C, D2.C, K1.A, K2.A
- net GND: now also MDL1.GND; no longer U$1.GND
- net GPIO0: now also MDL1.GPIO0; no longer U$1.GPIO0
- net GPIO14: now also MDL1.GPIO14; no longer U$1.GPIO14
- net GPIO16: now also MDL1.GPIO16; no longer U$1.GPIO16
- net GPIO4: now also MDL1.GPIO4, R6.1; no longer R3.1, U$1.GPIO4
- net GPIO5: now also MDL1.GPIO5, R3.1; no longer R6.1, U$1.GPIO5
- net RXD: now also MDL1.RXD; no longer U$1.RXD
- net TXD: now also MDL1.TXD; no longer U$1.TXD
Other:
- moved on the sheet: CONN-SW-1, CONN-SW-2, CONN-SW-3, R2, R5
